File: universal_fan_ctrl.kicad_pcb (KiCad board)
At the start: 2 copper layers, 13.6 x 11.6 mm, 14 parts, among them J1 Conn_01x03, J2 Conn_01x02, Q1 DMG3406L, U1 TLV76033DBZ, U2 ATtiny202-SS, U3 DS18B20

Commit message: Connected FAN_CTRL net to the spare AVR pin
Connections:
- U2 pad 4: unconnected-(U2-PA1-Pad4) -> /FAN_SW
Routing:
- net /FAN_SW: track 2.72 -> 8.01 mm
- net +3.3V: track 23.9 -> 25.0 mm
Changed lines of the file:
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@@
 	(net 6 "Net-(J1-Pin_1)")
 	(net 7 "Net-(J2-Pin_2)")
-	(net 8 "unconnected-(U2-PA1-Pad4)")
-	(net 9 "/MT")
-	(net 10 "/TR")
+	(net 8 "/MT")
+	(net 9 "/TR")
 	(footprint "Package_TO_SOT_SMD:SOT-23"
 		(layer "F.Cu")
@@
 			(layers "F.Cu" "F.Paste" "F.Mask")
 			(roundrect_rratio 0.25)
-			(net 10 "/TR")
+			(net 9 "/TR")
 			(pintype "passive")
 		)
@@
 			(layers "F.Cu" "F.Paste" "F.Mask")
 			(roundrect_rratio 0.25)
-			(net 10 "/TR")
+			(net 9 "/TR")
 			(pintype "passive")
 		)
@@
 			(layers "F.Cu" "F.Paste" "F.Mask")
 			(roundrect_rratio 0.25)
-			(net 9 "/MT")
+			(net 8 "/MT")
 			(pintype "passive")
 		)
@@
 			(layers "F.Cu" "F.Paste" "F.Mask")
 			(roundrect_rratio 0.25)
-			(net 9 "/MT")
+			(net 8 "/MT")
 			(pintype "passive")
 		)
@@
 			(layers "F.Cu" "F.Paste" "F.Mask")
 			(roundrect_rratio 0.25)
-			(net 8 "unconnected-(U2-PA1-Pad4)")
+			(net 3 "/FAN_SW")
 			(pinfunction "PA1")
 			(pintype "bidirectional")
@@
 			(layers "F.Cu" "F.Paste" "F.Mask")
 			(roundrect_rratio 0.25)
-			(net 9 "/MT")
+			(net 8 "/MT")
 			(pinfunction "PA2")
 			(pintype "bidirectional")
@@
 			(layers "F.Cu" "F.Paste" "F.Mask")
 			(roundrect_rratio 0.25)
-			(net 10 "/TR")
+			(net 9 "/TR")
 			(pinfunction "PA3")
 			(pintype "bidirectional")
@@
 	)
 	(segment
-		(start 147.5375 67.75)
-		(end 147.5375 71.7)
+		(start 147.15 67.75)
+		(end 146.46875 68.43125)
+		(width 0.2)
+		(layer "F.Cu")
+		(net 2)
+	)
+	(segment
+		(start 146.47375 72.805)
+		(end 146.46875 72.8)
 		(width 0.2)
 		(layer "F.Cu")
@@
 	)
 	(segment
-		(start 147.5375 72.4)
-		(end 147.9425 72.805)
+		(start 146.46875 72.8)
+		(end 146.46875 73.46875)
+		(width 0.2)
+		(layer "F.Cu")
+		(net 2)
+	)
+	(segment
+		(start 146.46875 68.43125)
+		(end 146.46875 72.8)
 		(width 0.2)
 		(layer "F.Cu")
@@
 	)
 	(segment
-		(start 146 73.9375)
-		(end 147.3 72.6375)
-		(width 0.2)
-		(layer "F.Cu")
-		(net 2)
-	)
-	(segment
-		(start 147.3 72.6375)
-		(end 147.5375 72.4)
+		(start 147.5375 67.75)
+		(end 147.15 67.75)
 		(width 0.2)
 		(layer "F.Cu")
@@
 	)
 	(segment
-		(start 147.9425 72.805)
-		(end 149.075 72.805)
+		(start 146 73.9375)
+		(end 146.46875 73.46875)
 		(width 0.2)
 		(layer "F.Cu")
@@
 	)
 	(segment
-		(start 147.5375 72.4)
-		(end 147.5375 71.7)
+		(start 149.075 72.805)
+		(end 146.47375 72.805)
 		(width 0.2)
 		(layer "F.Cu")
@@
 	)
 	(segment
+		(start 147.4 71)
+		(end 147.4 69.5)
+		(width 0.2)
+		(layer "F.Cu")
+		(net 3)
+	)
+	(segment
+		(start 147.905 68.995)
+		(end 149.075 68.995)
+		(width 0.2)
+		(layer "F.Cu")
+		(net 3)
+	)
+	(segment
+		(start 147.4 69.5)
+		(end 147.905 68.995)
+		(width 0.2)
+		(layer "F.Cu")
+		(net 3)
+	)
+	(segment
+		(start 147.935 71.535)
+		(end 147.4 71)
+		(width 0.2)
+		(layer "F.Cu")
+		(net 3)
+	)
+	(segment
 		(start 150.95 73.0375)
 		(end 150.95 72.65)
@@
 	)
 	(segment
+		(start 149.075 71.535)
+		(end 147.935 71.535)
+		(width 0.2)
+		(layer "F.Cu")
+		(net 3)
+	)
+	(segment
 		(start 150.95 72.65)
 		(end 149.835 71.535)
@@
 		(width 0.2)
 		(layer "F.Cu")
-		(net 9)
+		(net 8)
 	)
 	(segment
@@
 		(width 0.2)
 		(layer "F.Cu")
-		(net 9)
+		(net 8)
 	)
 	(segment
@@
 		(width 0.2)
 		(layer "F.Cu")
-		(net 9)
+		(net 8)
 	)
 	(segment
@@
 		(width 0.2)
 		(layer "F.Cu")
-		(net 9)
+		(net 8)
 	)
 	(segment
@@
 		(width 0.2)
 		(layer "F.Cu")
-		(net 9)
+		(net 8)
 	)
 	(segment
@@
 		(width 0.2)
 		(layer "F.Cu")
-		(net 9)
+		(net 8)
 	)
 	(segment
@@
 		(width 0.2)
 		(layer "F.Cu")
-		(net 10)
+		(net 9)
 	)
 	(segment
@@
 		(width 0.2)
 		(layer "F.Cu")
-		(net 10)
+		(net 9)
 	)
 	(segment
@@
 		(width 0.2)
 		(layer "F.Cu")
-		(net 10)
+		(net 9)
 	)
 	(segment
@@
 		(width 0.2)
 		(layer "F.Cu")
-		(net 10)
+		(net 9)
 	)
 	(segment
@@
 		(width 0.2)
 		(layer "F.Cu")
-		(net 10)
+		(net 9)
 	)
 	(segment
@@
 		(width 0.2)
 		(layer "F.Cu")
-		(net 10)
+		(net 9)
 	)
 	(segment
@@
 		(width 0.2)
 		(layer "F.Cu")
-		(net 10)
+		(net 9)
 	)
 	(segment
@@
 		(width 0.2)
 		(layer "F.Cu")
-		(net 10)
+		(net 9)
 	)
 	(zone

Commit message: kicad update, addressing #1
Parts:
- removed C1: 100n 35V, Resistor_SMD:R_0603_1608Metric
- removed R1: 100k, Resistor_SMD:R_0603_1608Metric
- added D2: BAT54J, Diode_SMD:D_SOD-323F, F.Cu at (149.3, 66.7)
- moved C2 1.70 mm to (147.6, 66.6)
- moved U1 1.70 mm to (144.9, 66.8)
- moved R4 0.95 mm to (142.2, 74.4)
- moved Rtr1 0.95 mm to (142.2, 75.9)
- moved R3 0.55 mm to (145.4, 74.4)
- moved Rmt1 0.55 mm to (145.4, 75.9)
- moved R5 0.40 mm to (147.8, 75.1)
Routing:
- net Net-(D2-K): track 16.8 -> 7.40 mm
- net /UPDI/~{RESET}: track 6.23 -> 3.23 mm
- net Net-(D2-A): track 2.26 -> 5.24 mm
- net +3.3V: track 25.0 -> 23.4 mm
- net /TR: track 6.39 -> 7.83 mm
- net GND: track 4.05 -> 5.11 mm
- net /MT: track 8.33 -> 9.05 mm
- added copper zone on B.Cu, net Net-(D2-K)
Other:
- board text added: "~{RST}/UPDI"
- board text removed: "~{RST}/PRG"
